Commit message: Three Robot

File: urdf/sly.urdf (robot description, URDF)
Before this commit: robot sly, 5 links, 4 joints
Links:
- link base_link: geometry collision mesh filename=package://sly_description/models/sly/meshes/base_link.STL; visual mesh filename=package://sly_description/models/sly/meshes/base_link.STL
- link wheel_0: geometry collision mesh filename=package://sly_description/models/sly/meshes/wheel_0.STL; visual mesh filename=package://sly_description/models/sly/meshes/wheel_0.STL
- link wheel_1: geometry collision mesh filename=package://sly_description/models/sly/meshes/wheel_1.STL; visual mesh filename=package://sly_description/models/sly/meshes/wheel_1.STL
- link wheel_2: geometry collision mesh filename=package://sly_description/models/sly/meshes/wheel_2.STL; visual mesh filename=package://sly_description/models/sly/meshes/wheel_2.STL
- link wheel_3: geometry collision mesh filename=package://sly_description/models/sly/meshes/wheel_3.STL; visual mesh filename=package://sly_description/models/sly/meshes/wheel_3.STL
